File: particle_photo_relay_board.sch (EAGLE design)
At the start: 12 parts, among them Q1 600mA/40V

Commit message: Add files via upload
P.R.A.C.C REV1 SCH and BRD files ready for review.
Parts:
- removed D3: GREEN, SparkFun-LED:LED-GREEN1206
- removed J1: (no value), SparkFun-Connectors:CONN_03SCREW
- removed J2, J3: (no value), SparkFun-Retired:CONN_023.5MM
- added C1, C2: 1uF, rcl:C-USC0805
- added J4, J5: (no value), SparkFun-Connectors:CONN_03-SCREW-5MM
- added R4, R7: 0, rcl:R-US_R0805
- added R5, R6: 0 - DNI, rcl:R-US_R0805
- added U2: MIC5219BM5, v-reg-micrel:MIC5219BM5
- R1: value (none) -> 330; device SparkFun-Resistors:RESISTORAXIAL-0.3 -> rcl:R-US_R0805
- R2, R3: value (none) -> 10; device SparkFun-Resistors:RESISTORAXIAL-0.3 -> rcl:R-US_R0805
- U$2: value RELAY-SPDT-2-G5V -> RELAYOMRON; device SparkFun-Retired:RELAY-SPDT-2-G5V -> Particle:RELAYOMRON
Connections:
- net N$5 renamed PHOTON_D7
- removed net N$10: J3.1, U$1.D1
- removed net N$6: J2.1, U$1.D0
- removed net N$7: J1.1, U$2.1
- removed net N$8: J1.3, U$2.10
- removed net N$9: J1.2, U$2.5, U$2.6
- removed net VCC: D2.A, R2.2
- new net 3V3_BACKUP: C2.1, R6.1, U2.OUT
- new net 3V3_PHOTON: R5.1, U$1.3V3
- new net COM: J4.2, U$2.MAIN
- new net NC: J4.3, U$2.NC
- new net NO: J4.1, U$2.NO
- new net PHOTON_D0: J5.2, U$1.D0
- new net PHOTON_D1: J5.3, U$1.D1
- new net VBUS_BACKUP: C1.1, R7.1, U2.IN
- new net VCOIL: D2.A, R2.2, R4.2, R5.2, R6.2
- new net VIN_PHOTON: R4.1, R7.2, U$1.VIN
- net GND: now also C1.2, C2.2, J5.1, U2.GND
- net N$1: now also U$2.COIL2; no longer U$2.9
- net N$2: now also U$2.COIL1; no longer U$2.2
Other:
- moved on the sheet: D1, D2, Q1, R1, R2, R3
